File: Hardware/PCB/Cansat_PCB_V1/untitled.kicad_sch (KiCad schematic)
At the start: 35 parts, among them IC1 Alim STM Baro GPS IMU, IC2 Alim STM Baro GPS IMU, J2 Connecteur Batterie, J3 Connecteur STLINK, J4 Connecteur Moteur, J5 Connecteur GPS, J6 Connecteur GPS, J7 Connecteur LoRa, U5 Alim 5V

Commit message: ajout 2 Led adr + btn cmd + buck LMR51625 => sch complet sans warnings et erreurs
Parts:
- removed C21: 0.1u, Capacitor_SMD:C_1210_3225Metric_Pad1.33x2.70mm_HandSolder, symbol Device:C_Small
- removed C22: 66u, Capacitor_SMD:C_0402_1005Metric_Pad0.74x0.62mm_HandSolder, symbol Device:C_Small
- removed C23: 2.2u, Capacitor_SMD:C_0402_1005Metric_Pad0.74x0.62mm_HandSolder, symbol Device:C_Small
- removed R20: 53.6k, Resistor_SMD:R_0402_1005Metric_Pad0.72x0.64mm_HandSolder, symbol Device:R_Small
- removed R22: 10.2k, Resistor_SMD:R_0402_1005Metric_Pad0.72x0.64mm_HandSolder, symbol Device:R_Small
- removed TP3: TestPoint, TestPoint:TestPoint_Pad_1.5x1.5mm, symbol Connector:TestPoint
- removed U5: Alim 5V, Package_TO_SOT_SMD:SOT-23-6, symbol Regulator_Switching:LMR51430
- added C31, C32: 100n, Capacitor_SMD:C_0402_1005Metric, symbol Device:C_Small
- added C33: 2.2u, Capacitor_SMD:C_0402_1005Metric_Pad0.74x0.62mm_HandSolder, symbol Device:C_Small
- added C34: 0.1u, Capacitor_SMD:C_1210_3225Metric_Pad1.33x2.70mm_HandSolder, symbol Device:C_Small
- added C35: 66u, Capacitor_SMD:C_0402_1005Metric_Pad0.74x0.62mm_HandSolder, symbol Device:C_Small
- added D4, D5: WS2812B-2020, LED_SMD:LED_WS2812B-2020_PLCC4_2.0x2.0mm, symbol LED:WS2812B-2020
- added R27: 10.2k, Resistor_SMD:R_0402_1005Metric_Pad0.72x0.64mm_HandSolder, symbol Device:R_Small
- added R28: 53.6k, Resistor_SMD:R_0402_1005Metric_Pad0.72x0.64mm_HandSolder, symbol Device:R_Small
- added TP5: TestPoint, TestPoint:TestPoint_Pad_1.5x1.5mm, symbol Connector:TestPoint
- added U5: LMR51625, Package_TO_SOT_SMD:SOT-23-6, symbol Homemade:LMR51430_1
- L1: footprint footprints:IND_WE-PD-SMT_7332_WRE -> (none)
Connections:
- net +3.3V: now also C31.1, C32.1, D4.4 (VDD), D5.4 (VDD)
- net +5V: now also C35.1, R28.2, TP5.1
- net GND: now also C31.2, C32.2, C33.2, C35.2, D4.2 (VSS), D5.2 (VSS), R27.2, U5.1 (GND)
- net VIN: now also C33.1, U5.3 (VIN), U5.5 (EN)
- net at L1.1: now also C34.2, U5.2 (SW)
- new net: D4.1 (DOUT), D5.3 (DIN)
- new net: R27.1, R28.1, U5.4 (FB)
- new net: C34.1, U5.6 (CB)
- new net LED_DATA: D4.3 (DIN)
- no-connect marks 7 -> 8
Other:
- note added: "LED Adressables"
- note added: "LEDs Commandables"
- note added: "découplage local"
- note added: "footprints : Package_TO_SOT_SMD:SOT-23-6"

Commit message: routage non fini : ceci est un commit de transfert de fichier vers un autre PC
Parts:
- renumbered D4 to D?, L1 to L?, TP1 to TP?, U5 to U?
Changed lines of the file:
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@@
 		(dnp no)
 		(fields_autoplaced yes)
-		(property "Reference" "#PWR043"
+		(property "Reference" "#PWR0101"
 			(at 36.83 88.9 0)
 			(effects
@@
 		)
 		(instances
-			(project ""
+			(project "Cansat_PCB"
 				(path "/43b9f51a-edfb-48c9-aab9-a28c7efe9297/24409c25-a13b-4fce-aa43-db656a14ada4"
-					(reference "#PWR043")
+					(reference "#PWR0101")
 					(unit 1)
 				)
@@
 		(dnp no)
 		(fields_autoplaced yes)
-		(property "Reference" "#PWR059"
+		(property "Reference" "#PWR0102"
 			(at 115.57 139.7 0)
 			(effects
@@
 		)
 		(instances
-			(project ""
+			(project "Cansat_PCB"
 				(path "/43b9f51a-edfb-48c9-aab9-a28c7efe9297/24409c25-a13b-4fce-aa43-db656a14ada4"
-					(reference "#PWR059")
+					(reference "#PWR0102")
 					(unit 1)
 				)
@@
 		(dnp no)
 		(fields_autoplaced yes)
-		(property "Reference" "D4"
+		(property "Reference" "D?"
 			(at 106.68 173.9198 0)
 			(effects
@@
 		)
 		(instances
-			(project ""
+			(project "Cansat_PCB"
 				(path "/43b9f51a-edfb-48c9-aab9-a28c7efe9297/24409c25-a13b-4fce-aa43-db656a14ada4"
-					(reference "D4")
+					(reference "D?")
 					(unit 1)
 				)
@@
 		(dnp no)
 		(fields_autoplaced yes)
-		(property "Reference" "L1"
+		(property "Reference" "L?"
 			(at 224.79 35.56 90)
 			(effects
@@
 		)
 		(instances
-			(project ""
+			(project "Cansat_PCB"
 				(path "/43b9f51a-edfb-48c9-aab9-a28c7efe9297/24409c25-a13b-4fce-aa43-db656a14ada4"
-					(reference "L1")
+					(reference "L?")
 					(unit 1)
 				)
@@
 		(dnp no)
 		(fields_autoplaced yes)
-		(property "Reference" "TP1"
+		(property "Reference" "TP?"
 			(at 32.258 175.26 90)
 			(effects
@@
 		)
 		(instances
-			(project ""
+			(project "Cansat_PCB"
 				(path "/43b9f51a-edfb-48c9-aab9-a28c7efe9297/24409c25-a13b-4fce-aa43-db656a14ada4"
-					(reference "TP1")
+					(reference "TP?")
 					(unit 1)
 				)
@@
 		(dnp no)
 		(fields_autoplaced yes)
-		(property "Reference" "U5"
+		(property "Reference" "U?"
 			(at 199.39 27.94 0)
 			(effects
@@
 		)
 		(instances
-			(project ""
+			(project "Cansat_PCB"
 				(path "/43b9f51a-edfb-48c9-aab9-a28c7efe9297/24409c25-a13b-4fce-aa43-db656a14ada4"
-					(reference "U5")
+					(reference "U?")
 					(unit 1)
 				)
@@
 		(dnp no)
 		(fields_autoplaced yes)
-		(property "Reference" "#PWR060"
+		(property "Reference" "#PWR0103"
 			(at 125.73 147.32 0)
 			(effects
@@
 		)
 		(instances
-			(project ""
+			(project "Cansat_PCB"
 				(path "/43b9f51a-edfb-48c9-aab9-a28c7efe9297/24409c25-a13b-4fce-aa43-db656a14ada4"
-					(reference "#PWR060")
+					(reference "#PWR0103")
 					(unit 1)
 				)

Commit message: nouvelles règles de routage Attention les pistes sont à l'ancienne taille : a corriger
Parts:
- removed TP2, TP?: TestPoint, TestPoint:TestPoint_Pad_1.5x1.5mm, symbol Connector:TestPoint
- added J8: connecteurb IHM, Connector_JST:JST_SH_BM04B-SRSS-TB_1x04-1MP_P1.00mm_Vertical, symbol Homemade:jst_4pin_with_mp
- added J9: Connecteur IHM, Connector_JST:JST_SH_BM04B-SRSS-TB_1x04-1MP_P1.00mm_Vertical, symbol Homemade:jst_4pin_with_mp
- added SW3: SW_Push, Button_Switch_SMD:SW_Push_1P1T_NO_CK_PTS125Sx43PSMTR, symbol Switch:SW_Push
- H1, H2, H3, H4: footprint customhole:mountinghole1.2mm -> footprints:mountinghole1.2mm
- J3: footprint footprints:SAMTEC_FTSH-107-01-L-DV-K-A -> footprints:FTSH-107-XX-YYY-DV-K; symbol FTSH-107-01-L-DV-K-A:FTSH-107-01-L-DV-K-A -> Homemade:FTSH-107-01-L-DV-K-A
- L1: renamed from L?; footprint (none) -> footprints:DFN6_3X3_STM
- gave numbers to parts that had none: 2
Connections:
- net +3.3V: now also J8.1 (Pin_1), J9.1 (Pin_1), SW3.1
- net GND: now also J8.4 (Pin_4), J8.MP, J9.4 (Pin_4), J9.MP
- net LED_DATA: now also J9.3 (Pin_3); no longer D4.3 (DIN)
- new net EXTI3: J9.2 (Pin_2)
- new net LED_DATA_IN: D4.3 (DIN), J8.3 (Pin_3)
- new net MainBTN: J8.2 (Pin_2), SW3.2
Other:
- note added: "Bouton de commande"
- note added: "Connecteurs IHM"
- note removed: "Connecteur USB"
- moved on the sheet: C27, C28, C31, C32, D3, D4, D5, IC2, J5, J6, J7, R24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

Commit message: Organisation des 6 couches + Placement des différents composants avant routage
Parts:
- IC2: value Alim STM Baro GPS IMU -> Alim LoRa
- J5: value Connecteur GPS -> Connecteur TOF
- L1: value 10u -> 4.7u; footprint footprints:DFN6_3X3_STM -> footprints:IND_WE-PD-SMT_7332_WRE
Changed lines of the file:
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@@
 			)
 		)
-		(property "Value" "Connecteur GPS"
+		(property "Value" "Connecteur TOF"
 			(at 114.935 133.35 0)
 			(effects
@@
 			)
 		)
-		(property "Value" "10u"
+		(property "Value" "4.7u"
 			(at 224.79 38.1 90)
 			(effects
@@
 			)
 		)
-		(property "Footprint" "footprints:DFN6_3X3_STM"
+		(property "Footprint" "footprints:IND_WE-PD-SMT_7332_WRE"
 			(at 224.79 40.64 0)
 			(effects
@@
 			)
 		)
-		(property "Datasheet" "~"
+		(property "Datasheet" "https://www.we-online.com/components/products/datasheet/74438356047.pdf"
 			(at 224.79 40.64 0)
 			(effects
@@
 			)
 		)
-		(property "Value" "Alim STM Baro GPS IMU"
+		(property "Value" "Alim LoRa"
 			(at 212.09 123.19 0)
 			(effects
