File: Hardware/PCB/Cansat_PCB_V2/Cansat_PCB.kicad_pcb (KiCad board)
At the start: 6 copper layers, 31.8 x 25.4 mm, 86 parts, among them IC1 Alim STM Baro GPS IMU, IC2 Alim LoRa, J1 Lecteur SD, J10 Connecteur IHM, J2 Connecteur Batterie, J3 Connecteur STLINK, J4 Connecteur Moteur, J5 Connecteur TOF, J6 Connecteur GPS, J7 Connecteur LoRa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

Commit message: ajout du logo vortex
Parts:
- added G***: LOGO, footprints:logo_cansat, F.Cu at (159.3, 101.0)
- added G***: LOGO, footprints:logo_cansat, B.Cu at (153.3, 96.2)
Other:
- board text added: "Cansat Vortex V2 Alexeï Douillard Amr Taouis Ares ENSEA"
- board text removed: "Cansat Vortex V2 Amr Taouis Alexeï Douillard Ares ENSEA"

Commit message: Logo update plus trace arragments
Parts:
- added G***: LOGO, footprints:logo_ENSEA, F.Cu at (137.8, 92.6)
- added G***: LOGO, footprints:logo_ARES, F.Cu at (140.1, 92.8)
- moved R20 1.20 mm to (158.5, 98.0), turned to 0 degrees
- moved G*** 0.47 mm to (158.9, 101.2)
- moved D1 0.22 mm to (138.2, 105.3)
- turned G*** to 180 degrees
Routing:
- net Net-(U2-PA11): track 5.27 -> 6.77 mm
- net Net-(U5-SW): track 8.75 -> 9.89 mm
- net CAM_EN: track 19.9 -> 19.0 mm
Other:
- board text added: "Cansat Vortex V2 Alexeï Douillard Amr Taouis ENSEA Ares"
- board text removed: "/"
- board text removed: "Cansat Vortex V2 Alexeï Douillard Amr Taouis Ares ENSEA"
