File: Hardware/PCB/Cansat_PCB_V3/Cansat_PCB_V3.kicad_sch (KiCad schematic)
At the start: 59 parts, among them J1 Lecteur SD, SW1 RSTBTN, SW2 boot, U1 Barometre BMP581, U2 STM32G431CBUx, U3 IMU BNO055, Y1 Crystal_GND24_Small, Y2 Oscillateur_IMU

Commit message: importing new readme
Other:
- title: CanSatv1 -> CanSatv3

Commit message: added the UART2 for the camera as well as M2 holes
Parts:
- removed R20: 10k, Resistor_SMD:R_0402_1005Metric_Pad0.72x0.64mm_HandSolder, symbol Device:R_Small
Connections:
- net ADC1_IN12_VBAT: now reaches U2.18 (PB1)
- net EXTI13_BTN: now reaches U2.2 (PC13)
- net ADC1_IN3_VBAT renamed USART2_TX_CAM
- net EXTI3_BTN renamed USART2_RX_CAM
- no-connect marks 11 -> 10
Other:
- moved on the sheet: D1, R7
Changed lines of the file:
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@@
 	(text "LED drivé à 1mA avec une tension de 2.2v ce qui \ndonne R=U/I=1.1kohms\nAttention la somme des courants sortant des GPIO \nne dois pas depasser 100mA"
 		(exclude_from_sim no)
-		(at 38.354 97.79 0)
+		(at 29.464 99.314 0)
 		(effects
 			(font
@@
 	)
 	(no_connect
-		(at 116.84 106.68)
+		(at 152.4 93.98)
 	)
 	(no_connect
@@
 		(at 373.38 156.21)
 	)
-	(no_connect
-		(at 116.84 93.98)
-	)
 	(wire
 		(pts
@@
 	(wire
 		(pts
-			(xy 91.44 104.14) (xy 87.63 104.14)
+			(xy 86.36 104.14) (xy 82.55 104.14)
 		)
 		(stroke
@@
 	(wire
 		(pts
-			(xy 152.4 93.98) (xy 154.94 93.98)
-		)
-		(stroke
-			(width 0)
-			(type default)
-		)
-	)
-	(wire
-		(pts
 			(xy 290.83 160.02) (xy 290.83 181.61)
 		)
@@
 	(wire
 		(pts
-			(xy 172.72 93.98) (xy 160.02 93.98)
-		)
-		(stroke
-			(width 0)
-			(type default)
-		)
-	)
-	(wire
-		(pts
 			(xy 285.75 182.88) (xy 285.75 176.53)
 		)
@@
 	(wire
 		(pts
-			(xy 96.52 104.14) (xy 99.06 104.14)
+			(xy 91.44 104.14) (xy 93.98 104.14)
 		)
 		(stroke
@@
 	(wire
 		(pts
-			(xy 106.68 104.14) (xy 116.84 104.14)
+			(xy 101.6 104.14) (xy 116.84 104.14)
 		)
 		(stroke
@@
 		)
 	)
+	(global_label "USART2_TX_CAM"
+		(shape input)
+		(at 152.4 71.12 0)
+		(fields_autoplaced yes)
+		(effects
+			(font
+				(size 1.27 1.27)
+			)
+			(justify left)
+		)
+		(property "Intersheetrefs" "${INTERSHEET_REFS}"
+			(at 170.3832 71.12 0)
+			(effects
+				(font
+					(size 1.27 1.27)
+				)
+				(justify left)
+				(hide yes)
+			)
+		)
+	)
 	(global_label "I2C3_SCL_IMU"
 		(shape input)
@@
 		)
 	)
-	(global_label "EXTI3_BTN"
-		(shape input)
-		(at 152.4 73.66 0)
-		(fields_autoplaced yes)
-		(effects
-			(font
-				(size 1.27 1.27)
-			)
-			(justify left)
-		)
-		(property "Intersheetrefs" "${INTERSHEET_REFS}"
-			(at 165.0613 73.66 0)
-			(effects
-				(font
-					(size 1.27 1.27)
-				)
-				(justify left)
-				(hide yes)
-			)
-		)
-	)
 	(global_label "SPI1_CS_SD"
 		(shape input)
@@
 		)
 	)
-	(global_label "ADC1_IN3_VBAT"
-		(shape input)
-		(at 152.4 71.12 0)
-		(fields_autoplaced yes)
-		(effects
-			(font
-				(size 1.27 1.27)
-			)
-			(justify left)
-		)
-		(property "Intersheetrefs" "${INTERSHEET_REFS}"
-			(at 169.7181 71.12 0)
-			(effects
-				(font
-					(size 1.27 1.27)
-				)
-				(justify left)
-				(hide yes)
-			)
-		)
-	)
 	(global_label "EXTI_BARO"
 		(shape input)
@@
 		)
 	)
-	(global_label "CAM_EN"
+	(global_label "TIM3_CHI_PWM4_MOT"
 		(shape input)
-		(at 172.72 93.98 0)
+		(at 116.84 86.36 180)
 		(fields_autoplaced yes)
 		(effects
@@
 				(size 1.27 1.27)
 			)
-			(justify left)
+			(justify right)
 		)
 		(property "Intersheetrefs" "${INTERSHEET_REFS}"
-			(at 182.9623 93.98 0)
+			(at 94.3816 86.36 0)
 			(effects
 				(font
 					(size 1.27 1.27)
 				)
-				(justify left)
+				(justify right)
 				(hide yes)
 			)
 		)
 	)
-	(global_label "TIM3_CHI_PWM4_MOT"
+	(global_label "USART2_RX_CAM"
 		(shape input)
-		(at 116.84 86.36 180)
+		(at 152.4 73.66 0)
 		(fields_autoplaced yes)
 		(effects
@@
 				(size 1.27 1.27)
 			)
-			(justify right)
+			(justify left)
 		)
 		(property "Intersheetrefs" "${INTERSHEET_REFS}"
-			(at 94.3816 86.36 0)
+			(at 170.6856 73.66 0)
 			(effects
 				(font
 					(size 1.27 1.27)
 				)
-				(justify right)
+				(justify left)
 				(hide yes)
 			)
@@
 		)
 	)
+	(global_label "ADC1_IN12_VBAT"
+		(shape input)
+		(at 116.84 106.68 180)
+		(fields_autoplaced yes)
+		(effects
+			(font
+				(size 1.27 1.27)
+			)
+			(justify right)
+		)
+		(property "Intersheetrefs" "${INTERSHEET_REFS}"
+			(at 98.3124 106.68 0)
+			(effects
+				(font
+					(size 1.27 1.27)
+				)
+				(justify right)
+				(hide yes)
+			)
+		)
+	)
 	(global_label "I2C1_SCL"
 		(shape input)
@@
 		)
 	)
+	(global_label "EXTI13_BTN"
+		(shape input)
+		(at 116.84 93.98 180)
+		(fields_autoplaced yes)
+		(effects
+			(font
+				(size 1.27 1.27)
+			)
+			(justify right)
+		)
+		(property "Intersheetrefs" "${INTERSHEET_REFS}"
+			(at 102.9692 93.98 0)
+			(effects
+				(font
+					(size 1.27 1.27)
+				)
+				(justify right)
+				(hide yes)
+			)
+		)
+	)
 	(global_label "NRST"
 		(shape input)
@@
 	(symbol
 		(lib_id "Device:LED")
-		(at 102.87 104.14 0)
+		(at 97.79 104.14 0)
 		(unit 1)
 		(exclude_from_sim no)
@@
 		(fields_autoplaced yes)
 		(property "Reference" "D1"
-			(at 101.2825 97.79 0)
+			(at 96.2025 97.79 0)
 			(effects
 				(font
@@
 		)
 		(property "Value" "LED"
-			(at 101.2825 100.33 0)
+			(at 96.2025 100.33 0)
 			(effects
 				(font
@@
 		)
 		(property "Footprint" "LED_SMD:LED_0603_1608Metric_Pad1.05x0.95mm_HandSolder"
-			(at 102.87 104.14 0)
+			(at 97.79 104.14 0)
 			(effects
 				(font
@@
 		)
 		(property "Datasheet" "~"
-			(at 102.87 104.14 0)
+			(at 97.79 104.14 0)
 			(effects
 				(font
@@
 		)
 		(property "Description" "Light emitting diode"
-			(at 102.87 104.14 0)
+			(at 97.79 104.14 0)
 			(effects
 				(font
@@
 		)
 		(property "Sim.Pins" "1=K 2=A"
-			(at 102.87 104.14 0)
+			(at 97.79 104.14 0)
 			(effects
 				(font
@@
 	(symbol
 		(lib_id "power:GND")
-		(at 87.63 104.14 270)
+		(at 82.55 104.14 270)
 		(unit 1)
 		(exclude_from_sim no)
@@
 		(fields_autoplaced yes)
 		(property "Reference" "#PWR017"
-			(at 81.28 104.14 0)
+			(at 76.2 104.14 0)
 			(effects
 				(font
@@
 		)
 		(property "Value" "GND"
-			(at 83.82 104.1399 90)
+			(at 78.74 104.1399 90)
 			(effects
 				(font
@@
 		)
 		(property "Footprint" ""
-			(at 87.63 104.14 0)
+			(at 82.55 104.14 0)
 			(effects
 				(font
@@
 		)
 		(property "Datasheet" ""
-			(at 87.63 104.14 0)
+			(at 82.55 104.14 0)
 			(effects
 				(font
@@
 		)
 		(property "Description" "Power symbol creates a global label with name \"GND\" , ground"
-			(at 87.63 104.14 0)
+			(at 82.55 104.14 0)
 			(effects
 				(font
@@
 	(symbol
 		(lib_id "Device:R_Small")
-		(at 93.98 104.14 90)
+		(at 88.9 104.14 90)
 		(unit 1)
 		(exclude_from_sim no)
@@
 		(on_board yes)
 		(dnp no)
-		(fields_autoplaced yes)
 		(property "Reference" "R7"
-			(at 93.98 99.06 90)
+			(at 88.646 99.822 90)
 			(effects
 				(font
@@
 		)
 		(property "Value" "1.1k"
-			(at 93.98 101.6 90)
+			(at 88.9 101.6 90)
 			(effects
 				(font
@@
 		)
 		(property "Footprint" "Resistor_SMD:R_0402_1005Metric_Pad0.72x0.64mm_HandSolder"
-			(at 93.98 104.14 0)
+			(at 88.9 104.14 0)
 			(effects
 				(font
@@
 		)
 		(property "Datasheet" "~"
-			(at 93.98 104.14 0)
+			(at 88.9 104.14 0)
 			(effects
 				(font
@@
 		)
 		(property "Description" "Resistor, small symbol"
-			(at 93.98 104.14 0)
+			(at 88.9 104.14 0)
 			(effects
 				(font
@@
 					(unit 1)
 				)
-			)
-		)
-	)
-	(symbol
-		(lib_id "Device:R_Small")
-		(at 157.48 93.98 270)
-		(unit 1)
-		(exclude_from_sim no)
-		(in_bom yes)
-		(on_board yes)
-		(dnp no)
-		(property "Reference" "R20"
-			(at 162.052 95.504 90)
-			(effects
-				(font
-					(size 1.27 1.27)
-				)
-			)
-		)
-		(property "Value" "10k"
-			(at 157.734 96.012 90)
-			(effects
-				(font
-					(size 1.27 1.27)
-				)
-			)
-		)
-		(property "Footprint" "Resistor_SMD:R_0402_1005Metric_Pad0.72x0.64mm_HandSolder"
-			(at 157.48 93.98 0)
-			(effects
-				(font
-					(size 1.27 1.27)
-				)
-				(hide yes)
-			)
-		)
-		(property "Datasheet" "~"
-			(at 157.48 93.98 0)
-			(effects
-				(font
-					(size 1.27 1.27)
-				)
-				(hide yes)
-			)
-		)
-		(property "Description" "Resistor, small symbol"
-			(at 157.48 93.98 0)
-			(effects
-				(font
-					(size 1.27 1.27)
-				)
-				(hide yes)
-			)
-		)
-		(pin "1"
-		)
-		(pin "2"
-		)
-		(instances
-			(project "Cansat_PCB_V3"
-				(path "/43b9f51a-edfb-48c9-aab9-a28c7efe9297"
-					(reference "R20")
-					(unit 1)
-				)
