File: Hardware/PCB/Cansat_PCB_V3/connectique_et_alimentation.kicad_sch (KiCad schematic)
At the start: 38 parts, among them IC1 Alim STM Baro GPS IMU, IC2 Alim LoRa, J10 Connecteur IHM, J2 Connecteur Batterie, J3 Connecteur STLINK, J4 Connecteur Moteur, J5 Connecteur TOF, J6 Connecteur GPS, J7 Connecteur LoRa, J8 Connecteur Camera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

Commit message: importing new readme
Other:
- title: CanSatv1 -> CanSatv3

Commit message: added the UART2 for the camera as well as M2 holes
Parts:
- removed J8: Connecteur Camera, Connector_JST:JST_SH_BM02B-SRSS-TB_1x02-1MP_P1.00mm_Vertical, symbol Connector:Conn_01x02_Pin
- added J9: Connecteur Camera, Connector_JST:JST_SH_BM04B-SRSS-TB_1x04-1MP_P1.00mm_Vertical, symbol Homemade:jst_4pin_with_mp
- H1, H2, H3, H4: footprint footprints:mountinghole1.2mm -> MountingHole:MountingHole_2.2mm_M2_ISO7380_Pad
Connections:
- net +3.3V: now also J9.1 (Pin_1)
- net GND: now also J9.4 (Pin_4), J9.MP
- net ADC1_IN3_VBAT renamed ADC1_IN12_VBAT
- net EXTI3_BTN renamed EXTI13_BTN
- new net USART2_RX_CAM: J9.2 (Pin_2)
- new net USART2_TX_CAM: J9.3 (Pin_3)

Commit message: mega big readme update for the mechanical and wind tunnel parts
Parts:
- F1: value Littel fuse 435 1.25A -> Littel fuse 435 1.5A
Changed lines of the file:
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@@
 			)
 		)
-		(property "Value" "Littel fuse 435 1.25A"
+		(property "Value" "Littel fuse 435 1.5A"
 			(at 164.592 37.592 0)
 			(effects
